Commit message: PR2: frames (F8), calibration (F2-F5, A'), G2 and G4
frames/      FrameNames, TiltMeasurement, GravityAlignedWorldFrame (F8 as a
             ReferenceFrame node), PelvisFrameTriad (the §13 hazard as a chain).
calibration/ CaptureSet, BaseInitializer (F2 + gauge tracking), BootstrapSolver
             (F3), MarkerLayoutSolver (F4), BaseAlignmentSolver (F5),
             AlternatingCalibrator (A'), CalibrationReport.
gates/       BootstrapSpreadGate (G2), HeldOutResidualGate (G4). Neither imports
             calibration; both take their inputs at construction.
core/        ObservationModel -- §0's equation, written once and shared by
             calibration, gates and later runtime.

Plant-and-recover is green: noiseless K=5 recovers layouts and base poses to
4.6e-15 m, J is monotone across every half-step, 20% occlusion is handled, and
K_ij bookkeeping is asserted.

Five things found by building it, each documented at the code:

1. An exact gauge freedom. Delta -> Delta*G for a pure translation g shifts every
   layout by R_i(q)^T g, which is a symmetry when g lies along an axis every
   marked link only rotates about. The toy's hip and knee both pitched about y,
   so A' converged to J=7.6e-29 -- machine zero -- and landed 13 mm from truth
   with every cluster displaced identically. The hip now rolls about x.

2. The cluster frame must be centred on the gauge markers' centroid. Using their
   raw positions puts c at the world origin, so Delta carries metres and F2's
   Delta = I is nowhere near the solution; A' then settles in a local minimum
   2 m out, monotonically.

3. Layout accuracy is not sigma/sqrt(K). It is dominated by the gauge cluster's
   angular error sigma/(sqrt(N) r_perp) times the lever arm to each link.
   Measured: clean the gauge markers and error is 0.089 mm at K=30 scaling as a
   clean 1/sqrt(K); leave them noisy and it is 0.383 mm scaling as K^-0.25,
   because the reference shape comes from one capture and that noise never
   averages. PR_PLAN's 0.2 mm target is unreachable for that reason, not for an
   implementation one. Thresholds set from the measured decomposition.

4. G2's expected spread has to include that gauge term, per marker and per lever
   arm, or the gate fires on clean data. And correlating the deviation MAGNITUDE
   finds nothing -- it is V-shaped in the joint angle; signed components find the
   offending joint.

5. G4 does not show PR_PLAN's asymmetry. An i.i.d. split shares a systematic
   bias equally, so in-sample and held-out rise together (within 3%). Held-out
   validation detects overfitting, and 90 parameters against 1680 observations
   have nothing to overfit. The absolute level, not the ratio, is the signal.

Co-Authored-By: Claude Opus 5 (1M context) <noreply@anthropic.com>
Claude-Session: https://claude.ai/code/session_01PF5WeJiuCwXD6o8wVt7oA5

File: src/test/resources/us/ihmc/alexMocap/model/toy6dof.urdf (robot description, URDF)
Before this commit: robot toy6dof, 7 links, 6 joints
Joints:
- joint l_ankle: axis 1 0 0 -> 0 1 0
- joint l_hip: axis 0 1 0 -> 1 0 0
- joint r_ankle: axis 1 0 0 -> 0 1 0
- joint r_hip: axis 0 1 0 -> 1 0 0
